File: bandpass_filter_design/bandpass_filter_design.kicad_pcb (KiCad board)
At the start: 2 copper layers, 154.3 x 47.6 mm, 45 parts, among them J1 Conn_Coaxial, J2 Conn_01x09_Male, J3 Conn_Coaxial

Commit message: Prerefactor
Parts:
- added C19: 0,5pF, Capacitor_SMD:C_0805_2012Metric_Pad1.15x1.40mm_HandSolder, F.Cu at (92.4, 83.8)
- added C20: 0,5pF, Capacitor_SMD:C_0805_2012Metric_Pad1.15x1.40mm_HandSolder, F.Cu at (193.2, 85.3)
- added G***: LOGO, digital_capacitors:open-source-logo-2, F.Cu at (204.5, 102.9)
- C16, C3: value 10pF -> 7,5pF
- C18: value 0.5pF -> 0,5pF
- moved C18 4.34 mm to (197.4, 85.3)
Connections:
- C18 pad 2: Net-(C12-Pad8) -> Net-(C18-Pad2)
- C2 pad 1: Net-(C1-Pad10) -> Net-(C19-Pad2)
Routing:
- net Net-(C18-Pad2): track 0.00 -> 2.13 mm
- net Net-(C19-Pad2): track 0.00 -> 2.00 mm
- net Net-(C1-Pad10): track 54.6 -> 53.7 mm
- net Net-(C16-Pad2): track 10.5 -> 9.62 mm

Commit message: Big refactor and updated FFT sink look
Parts:
- removed G***: LOGO, digital_capacitors:open-source-logo-2
- removed R1, R19, R2, R20, R21, R3: 7,5k, Resistor_SMD:R_0805_2012Metric_Pad1.15x1.40mm_HandSolder
- removed R10, R12, R13, R14, R15, R16, R17, R5, R6, R7, R8, R9: 2,7k, Resistor_SMD:R_0805_2012Metric_Pad1.15x1.40mm_HandSolder
- added D1: BZX84Cxx, Diode_SMD:D_SOT-23_ANK, B.Cu at (133.0, 99.1)
- added D2: BZX84Cxx, Diode_SMD:D_SOT-23_ANK, B.Cu at (128.8, 98.8)
- added D3: BZX84Cxx, Diode_SMD:D_SOT-23_ANK, F.Cu at (130.6, 112.0)
- added D4: BZX84Cxx, Diode_SMD:D_SOT-23_ANK, B.Cu at (125.0, 99.1)
- added D5: BZX84Cxx, Diode_SMD:D_SOT-23_ANK, B.Cu at (120.7, 99.2)
- added R22: 7.5R, Resistor_SMD:R_0805_2012Metric_Pad1.15x1.40mm_HandSolder, B.Cu at (132.0, 103.0)
- added R23: 7.5R, Resistor_SMD:R_0805_2012Metric_Pad1.15x1.40mm_HandSolder, B.Cu at (127.8, 102.9)
- added R24: 7.5R, Resistor_SMD:R_0805_2012Metric_Pad1.15x1.40mm_HandSolder, F.Cu at (126.5, 112.1)
- added R25: 7.5R, Resistor_SMD:R_0805_2012Metric_Pad1.15x1.40mm_HandSolder, B.Cu at (124.0, 103.0)
- added R26: 7.5R, Resistor_SMD:R_0805_2012Metric_Pad1.15x1.40mm_HandSolder, B.Cu at (119.6, 103.0)
- moved L2 0.51 mm to (131.6, 87.9)
Connections:
- C1 pad 1: Net-(C1-Pad1) -> /ENser
- C1 pad 12: Net-(C1-Pad12) -> /DATA
- C1 pad 3: Net-(C1-Pad3) -> /CLK
- C11 pad 5: Net-(C11-Pad5) -> /CLK
- C11 pad 6: Net-(C11-Pad6) -> /ENinv_1
- C11 pad 7: Net-(C11-Pad7) -> /DATA
- C12 pad 5: Net-(C12-Pad5) -> /CLK
- C12 pad 6: Net-(C12-Pad6) -> /ENinv_2
- C12 pad 7: Net-(C12-Pad7) -> /DATA
- C17 pad 1: Net-(C17-Pad1) -> /ENser
- C17 pad 12: Net-(C17-Pad12) -> /DATA
- C17 pad 3: Net-(C17-Pad3) -> /CLK
- C7 pad 5: Net-(C7-Pad5) -> /CLK
- C7 pad 6: Net-(C7-Pad6) -> /ENinv_1
- C7 pad 7: Net-(C7-Pad7) -> /DATA
- C8 pad 5: Net-(C8-Pad5) -> /CLK
- C8 pad 6: Net-(C8-Pad6) -> /ENinv_2
- C8 pad 7: Net-(C8-Pad7) -> /DATA
- J2 pad 1: /DATA -> Net-(J2-Pad1)
- J2 pad 2: /CLK -> Net-(J2-Pad2)
- J2 pad 3: /ENser -> Net-(J2-Pad3)
- J2 pad 4: /ENinv_1 -> Net-(J2-Pad4)
- J2 pad 5: /ENinv_2 -> Net-(J2-Pad5)
Routing:
- net /DATA: track 243.8 -> 223.3 mm, vias 3 -> 9
- net /ENinv_1: track 60.5 -> 76.5 mm, vias 4 -> 8
- net /CLK: track 219.0 -> 233.6 mm, vias 5 -> 13
- net /ENser: track 188.7 -> 174.1 mm, vias 2 -> 4
- net /ENinv_2: track 84.9 -> 93.5 mm, vias 5 -> 7
- net Net-(C1-Pad12): track 7.09 -> 0.00 mm, vias 1 -> 0
- net Net-(C11-Pad5): track 7.01 -> 0.00 mm, vias 1 -> 0
- net Net-(C8-Pad7): track 6.89 -> 0.00 mm, vias 1 -> 0
- net Net-(C12-Pad7): track 6.63 -> 0.00 mm, vias 1 -> 0
- net Net-(C17-Pad12): track 6.23 -> 0.00 mm, vias 1 -> 0
- net Net-(C7-Pad5): track 6.20 -> 0.00 mm, vias 1 -> 0
- net Net-(C12-Pad5): track 6.20 -> 0.00 mm, vias 1 -> 0
- net Net-(C1-Pad3): track 5.97 -> 0.00 mm, vias 1 -> 0
- net Net-(C17-Pad3): track 5.95 -> 0.00 mm, vias 1 -> 0
- net Net-(C8-Pad5): track 5.38 -> 0.00 mm, vias 1 -> 0
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- added copper zone on B.Cu, net GND
Other:
- board size 154.3 x 47.6 mm -> 152.4 x 48.3 mm

Commit message: Pre-module commit
Parts:
- added J4: Conn_01x02_Male, Connector_PinHeader_2.54mm:PinHeader_1x02_P2.54mm_Vertical, F.Cu at (72.1, 97.9)
- added J5: Conn_01x02_Male, Connector_PinHeader_2.54mm:PinHeader_1x02_P2.54mm_Vertical, F.Cu at (208.5, 98.0)
- J1, J3: footprint digital_capacitors:SMA_Amphenol_901-144_Vertical -> Connector_Coaxial:SMA_Amphenol_901-144_Vertical
- L1, L2, L3: footprint Inductor_SMD:L_0603_1608Metric_Pad1.05x0.95mm_HandSolder -> Inductor_SMD:L_0402_1005Metric
- turned C8 to 90 degrees
- turned C11 to 0 degrees
- turned C12 to 90 degrees
- turned C7 to 0 degrees
Connections:
- net Net-(C16-Pad1) renamed /SIG_OUT
- net Net-(C3-Pad2) renamed /SIG_IN
Routing:
- net /SIG_IN: track 7.62 -> 24.3 mm
- net /SIG_OUT: track 7.37 -> 23.6 mm
- net /ENinv_1: track 76.5 -> 79.3 mm
- net /DATA: track 223.3 -> 226.0 mm
- net GND: track 28.1 -> 25.7 mm
- net /CLK: track 233.6 -> 235.9 mm
- net /ENinv_2: track 93.5 -> 94.7 mm
- net Net-(C12-Pad8): track 62.0 -> 62.6 mm
