File: bandpass_filter_design/bandpass_filter_design.sch (KiCad schematic (older format))
At the start: 12 parts

Commit message: Bandpass filter done
Parts:
- removed C?: CP1, symbol Device:CP1
- added C1, C17: PE64102, digital_capacitors:PE64102-QFN, symbol digital_capacitors:PE64102
- added C13, C4: 1.8pF, Capacitor_SMD:C_0805_2012Metric_Pad1.15x1.40mm_HandSolder, symbol Device:CP1
- added C14: 15pF, Capacitor_SMD:C_0805_2012Metric_Pad1.15x1.40mm_HandSolder, symbol Device:CP1
- added C16, C3: 10pF, Capacitor_SMD:C_0805_2012Metric_Pad1.15x1.40mm_HandSolder, symbol Device:CP1
- added C18: 0.5pF, Capacitor_SMD:C_0805_2012Metric_Pad1.15x1.40mm_HandSolder, symbol Device:CP1
- added C2: 0,5pF, Capacitor_SMD:C_0805_2012Metric_Pad1.15x1.40mm_HandSolder, symbol Device:CP1
- added J2: Conn_01x09_Male, Connector_PinHeader_2.54mm:PinHeader_1x09_P2.54mm_Vertical, symbol Connector:Conn_01x09_Male
- added L1, L2, L3: 4nH, Inductor_SMD:L_0603_1608Metric_Pad1.05x0.95mm_HandSolder, symbol Device:L
- added R1, R19, R2, R20, R21, R3: 7,5k, Resistor_SMD:R_0805_2012Metric_Pad1.15x1.40mm_HandSolder, symbol Device:R
- added R10, R12, R13, R14, R15, R16, R17, R5, R6, R7, R8, R9: 2,7k, Resistor_SMD:R_0805_2012Metric_Pad1.15x1.40mm_HandSolder, symbol Device:R
- added R11, R18, R4: 68k, Resistor_SMD:R_0805_2012Metric_Pad1.15x1.40mm_HandSolder, symbol Device:R
- C10, C15, C6: renamed from C?; footprint (none) -> digital_capacitors:NCD2100-TSOT-6
- C11, C12, C7, C8: renamed from C?; footprint (none) -> digital_capacitors:PE64909-QFN
- C5: renamed from C?; value CP1 -> 15pF; footprint (none) -> Capacitor_SMD:C_0805_2012Metric_Pad1.15x1.40mm_HandSolder
- C9: renamed from C?; value CP1 -> 18pF; footprint (none) -> Capacitor_SMD:C_0805_2012Metric_Pad1.15x1.40mm_HandSolder
- J1, J3: renamed from J?; footprint (none) -> Connector_Coaxial:SMA_Amphenol_901-144_Vertical
Connections:
- net labels added: CLK, DATA, ENinv_1, ENinv_2, ENser, VDD, ~ENmid, ~ENres
- wire segments 49 -> 263
Other:
- moved on the sheet: C10, C11, C15, C5, C6, C7, C8, C9, J1, J3

Commit message: Prerefactor
Parts:
- added C19, C20: 0,5pF, Capacitor_SMD:C_0805_2012Metric_Pad1.15x1.40mm_HandSolder, symbol Device:CP1
- C16, C3: value 10pF -> 7,5pF
- C18: value 0.5pF -> 0,5pF
Connections:
- net at C1.10 (RF+), C1.9 (RF+), C4.1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: now also C19.1; no longer C2.1
- net at C12.8 (RF+), C12.9 (RF+), C13.1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: now also C20.2; no longer C18.2
- new net: C19.2, C2.1
- new net: C18.2, C20.1
Other:
- moved on the sheet: C18, C2
Changed lines of the file:
@@
-$EndComp
-$Comp
-L digital_capacitors:PE64102 C1
-U 1 1 5C65588C
-P 2475 3050
-F 0 "C1" H 2475 3615 50  0000 C CNN
-F 1 "PE64102" H 2475 3524 50  0000 C CNN
-F 2 "digital_capacitors:PE64102-QFN" H 2525 3150 50  0001 C CNN
-F 3 "https://www.psemi.com/pdf/datasheets/pe64102ds.pdf" H 2525 3150 50  0001 C CNN
-	1    2475 3050
-	1    0    0    -1
 $EndComp
 $Comp
 L Device:CP1 C2
 U 1 1 5C65D3DF
-P 2475 3750
-F 0 "C2" V 2715 3750 50  0000 C CNN
-F 1 "0,5pF" V 2615 3750 50  0000 C CNN
-F 2 "Capacitor_SMD:C_0805_2012Metric_Pad1.15x1.40mm_HandSolder" H 2475 3750 50  0001 C CNN
-F 3 "~" H 2475 3750 50  0001 C CNN
-	1    2475 3750
+P 2275 3750
+F 0 "C2" V 2515 3750 50  0000 C CNN
+F 1 "0,5pF" V 2415 3750 50  0000 C CNN
+F 2 "Capacitor_SMD:C_0805_2012Metric_Pad1.15x1.40mm_HandSolder" H 2275 3750 50  0001 C CNN
+F 3 "~" H 2275 3750 50  0001 C CNN
+	1    2275 3750
 	0    1    1    0
 $EndComp
@@
 P 1350 3450
 F 0 "C3" V 1098 3450 50  0000 C CNN
-F 1 "10pF" V 1189 3450 50  0000 C CNN
+F 1 "7,5pF" V 1189 3450 50  0000 C CNN
 F 2 "Capacitor_SMD:C_0805_2012Metric_Pad1.15x1.40mm_HandSolder" H 1350 3450 50  0001 C CNN
 F 3 "~" H 1350 3450 50  0001 C CNN
@@
 	0    1    1    0
 $EndComp
-Wire Wire Line
-	2975 3750 2625 3750
-$Comp
-L digital_capacitors:PE64102 C17
-U 1 1 5C666B44
-P 9300 2950
-F 0 "C17" H 9300 3515 50  0000 C CNN
-F 1 "PE64102" H 9300 3424 50  0000 C CNN
-F 2 "digital_capacitors:PE64102-QFN" H 9350 3050 50  0001 C CNN
-F 3 "https://www.psemi.com/pdf/datasheets/pe64102ds.pdf" H 9350 3050 50  0001 C CNN
-	1    9300 2950
-	1    0    0    -1
-$EndComp
 $Comp
 L Device:CP1 C18
 U 1 1 5C666B4B
-P 9300 3550
-F 0 "C18" V 9530 3550 50  0000 C CNN
-F 1 "0.5pF" V 9450 3550 50  0000 C CNN
-F 2 "Capacitor_SMD:C_0805_2012Metric_Pad1.15x1.40mm_HandSolder" H 9300 3550 50  0001 C CNN
-F 3 "~" H 9300 3550 50  0001 C CNN
-	1    9300 3550
+P 9550 3550
+F 0 "C18" V 9780 3550 50  0000 C CNN
+F 1 "0,5pF" V 9700 3550 50  0000 C CNN
+F 2 "Capacitor_SMD:C_0805_2012Metric_Pad1.15x1.40mm_HandSolder" H 9550 3550 50  0001 C CNN
+F 3 "~" H 9550 3550 50  0001 C CNN
+	1    9550 3550
 	0    1    1    0
 $EndComp
@@
 P 10350 2850
 F 0 "C16" V 10098 2850 50  0000 C CNN
-F 1 "10pF" V 10189 2850 50  0000 C CNN
+F 1 "7,5pF" V 10189 2850 50  0000 C CNN
 F 2 "Capacitor_SMD:C_0805_2012Metric_Pad1.15x1.40mm_HandSolder" H 10350 2850 50  0001 C CNN
 F 3 "~" H 10350 2850 50  0001 C CNN
@@
 	8250 3750 8250 3250
 Wire Wire Line
-	9450 3550 9900 3550
-Wire Wire Line
 	2875 2750 2925 2750
 Wire Wire Line
 	2925 2750 2925 2850
 Wire Wire Line
-	2925 3150 2875 3150
-Wire Wire Line
-	2875 3050 2925 3050
-Connection ~ 2925 3050
-Wire Wire Line
-	2925 3050 2925 3150
-Wire Wire Line
-	2875 2950 2925 2950
-Connection ~ 2925 2950
-Wire Wire Line
-	2925 2950 2925 3050
-Wire Wire Line
 	2875 2850 2925 2850
-Connection ~ 2925 2850
-Wire Wire Line
-	2925 2850 2925 2950
-Wire Wire Line
-	2875 3250 2975 3250
-Wire Wire Line
-	2875 3350 2975 3350
-Wire Wire Line
-	2975 3350 2975 3250
-Connection ~ 2975 3350
-Wire Wire Line
-	2975 3750 2975 3350
 Wire Wire Line
 	4350 2100 4350 2050
@@
 	9750 2650 9750 2750
 Wire Wire Line
-	9750 3050 9700 3050
-Wire Wire Line
-	9700 2950 9750 2950
-Connection ~ 9750 2950
-Wire Wire Line
-	9750 2950 9750 3050
-Wire Wire Line
-	9700 2850 9750 2850
-Connection ~ 9750 2850
-Wire Wire Line
-	9750 2850 9750 2950
-Wire Wire Line
 	9700 2750 9750 2750
-Connection ~ 9750 2750
-Wire Wire Line
-	9750 2750 9750 2850
-Wire Wire Line
-	9700 3150 9900 3150
-Wire Wire Line
-	9900 3150 9900 3250
-Wire Wire Line
-	9700 3250 9900 3250
-Connection ~ 9900 3250
-Wire Wire Line
-	9900 3250 9900 3550
-Wire Wire Line
-	9900 3150 9900 2850
-Wire Wire Line
-	9900 2850 10200 2850
-Connection ~ 9900 3150
 Wire Wire Line
 	6800 2100 6800 2000
@@
 VDD
 Wire Wire Line
-	2075 2750 2025 2750
-Wire Wire Line
-	1725 3750 2325 3750
-Wire Wire Line
-	2075 2850 2025 2850
-Wire Wire Line
-	2025 2850 2025 2750
-Connection ~ 2025 2750
-Wire Wire Line
-	2025 2750 1725 2750
-Wire Wire Line
 	8600 2650 8850 2650
 Wire Wire Line
@@
 Wire Wire Line
 	8850 2650 8900 2650
-Wire Wire Line
-	8600 3550 9150 3550
 $Comp
 L power:PWR_FLAG #FLG01
@@
 DATA
 Wire Wire Line
-	2075 3150 1925 3150
-Wire Wire Line
-	1925 3150 1925 3875
-Wire Wire Line
 	2050 4250 2200 4250
 Wire Wire Line
 	2050 3875 2050 3250
-Wire Wire Line
-	2050 3250 2075 3250
-Wire Wire Line
-	1800 3875 1800 3050
-Wire Wire Line
-	1800 3050 2075 3050
 $Comp
 L Device:R R19
@@
 Wire Wire Line
 	5450 1950 5450 2100
-Connection ~ 2975 3250
 Wire Wire Line
 	8600 2650 8600 3250
@@
 Wire Wire Line
 	9850 3375 9850 4000
-Wire Wire Line
-	2975 3250 3120 3250
 Wire Wire Line
 	1500 3450 1725 3450
@@
 	1725 3450 1725 3750
 Wire Wire Line
-	1725 2750 1725 3450
-Wire Wire Line
 	8250 3250 8600 3250
 Connection ~ 8250 3250
@@
 Wire Wire Line
 	8600 3250 8600 3550
+Wire Wire Line
+	9900 2850 10200 2850
+Wire Wire Line
+	9700 2850 9750 2850
+Connection ~ 9750 2750
+Wire Wire Line
+	9750 2750 9750 2850
+Wire Wire Line
+	9900 3250 9900 3550
+Connection ~ 9900 3250
+Wire Wire Line
+	9700 3250 9900 3250
+Wire Wire Line
+	9900 3150 9900 2850
+Wire Wire Line
+	9900 3150 9900 3250
+Connection ~ 9900 3150
+Wire Wire Line
+	9700 3150 9900 3150
+Wire Wire Line
+	9750 3050 9700 3050
+Wire Wire Line
+	9700 2950 9750 2950
+Wire Wire Line
+	9750 2950 9750 3050
+Connection ~ 9750 2950
+Connection ~ 9750 2850
+Wire Wire Line
+	9750 2850 9750 2950
+$Comp
+L digital_capacitors:PE64102 C17
+U 1 1 5C666B44
+P 9300 2950
+F 0 "C17" H 9300 3515 50  0000 C CNN
+F 1 "PE64102" H 9300 3424 50  0000 C CNN
+F 2 "digital_capacitors:PE64102-QFN" H 9350 3050 50  0001 C CNN
+F 3 "https://www.psemi.com/pdf/datasheets/pe64102ds.pdf" H 9350 3050 50  0001 C CNN
+	1    9300 2950
+	1    0    0    -1
+$EndComp
+Wire Wire Line
+	2975 3250 3120 3250
+Connection ~ 2975 3250
+Wire Wire Line
+	1725 2750 1725 3450
+Wire Wire Line
+	2025 2750 1725 2750
+Wire Wire Line
+	2075 2850 2025 2850
+Wire Wire Line
+	2025 2850 2025 2750
+Connection ~ 2025 2750
+Wire Wire Line
+	2075 2750 2025 2750
+Wire Wire Line
+	2050 3250 2075 3250
+Wire Wire Line
+	1800 3050 2075 3050
+Wire Wire Line
+	1925 3150 1925 3875
+Wire Wire Line
+	2075 3150 1925 3150
+Wire Wire Line
+	1800 3875 1800 3050
+Wire Wire Line
+	2975 3750 2975 3350
+Wire Wire Line
+	2975 3350 2975 3250
+Connection ~ 2975 3350
+Wire Wire Line
+	2875 3350 2975 3350
+Wire Wire Line
+	2875 3250 2975 3250
+Wire Wire Line
+	2875 3050 2925 3050
+Wire Wire Line
+	2875 2950 2925 2950
+Connection ~ 2925 2850
+Wire Wire Line
+	2925 2850 2925 2950
+Connection ~ 2925 2950
+Wire Wire Line
+	2925 2950 2925 3050
+Wire Wire Line
+	2925 3150 2875 3150
+Connection ~ 2925 3050
+Wire Wire Line
+	2925 3050 2925 3150
+$Comp
+L digital_capacitors:PE64102 C1
+U 1 1 5C65588C
+P 2475 3050
+F 0 "C1" H 2475 3615 50  0000 C CNN
+F 1 "PE64102" H 2475 3524 50  0000 C CNN
+F 2 "digital_capacitors:PE64102-QFN" H 2525 3150 50  0001 C CNN
+F 3 "https://www.psemi.com/pdf/datasheets/pe64102ds.pdf" H 2525 3150 50  0001 C CNN
+	1    2475 3050
+	1    0    0    -1
+$EndComp
+$Comp
+L Device:CP1 C19
+U 1 1 5C8125A4
+P 2700 3750
+F 0 "C19" V 2940 3750 50  0000 C CNN
+F 1 "0,5pF" V 2840 3750 50  0000 C CNN
+F 2 "Capacitor_SMD:C_0805_2012Metric_Pad1.15x1.40mm_HandSolder" H 2700 3750 50  0001 C CNN
+F 3 "~" H 2700 3750 50  0001 C CNN
+	1    2700 3750
+	0    1    1    0
+$EndComp
+Wire Wire Line
+	1725 3750 2125 3750
+Wire Wire Line
+	2425 3750 2550 3750
+Wire Wire Line
+	2850 3750 2975 3750
+$Comp
+L Device:CP1 C20
+U 1 1 5C871ABB
+P 9250 3550
+F 0 "C20" V 9480 3550 50  0000 C CNN
+F 1 "0,5pF" V 9400 3550 50  0000 C CNN
+F 2 "Capacitor_SMD:C_0805_2012Metric_Pad1.15x1.40mm_HandSolder" H 9250 3550 50  0001 C CNN
+F 3 "~" H 9250 3550 50  0001 C CNN
+	1    9250 3550
+	0    1    1    0
+$EndComp
+Wire Wire Line
+	9100 3550 8600 3550
+Wire Wire Line
+	9700 3550 9900 3550
 $EndSCHEMATC

Commit message: Big refactor and updated FFT sink look
Parts:
- removed R1, R19, R2, R20, R21, R3: 7,5k, Resistor_SMD:R_0805_2012Metric_Pad1.15x1.40mm_HandSolder, symbol Device:R
- removed R10, R12, R13, R14, R15, R16, R17, R5, R6, R7, R8, R9: 2,7k, Resistor_SMD:R_0805_2012Metric_Pad1.15x1.40mm_HandSolder, symbol Device:R
- added D1, D2, D3, D4, D5: BZX84Cxx, Diode_SMD:D_SOT-23_ANK, symbol Diode:BZX84Cxx
- added R22, R23, R24, R25, R26: 7.5R, Resistor_SMD:R_0805_2012Metric_Pad1.15x1.40mm_HandSolder, symbol Device:R
Connections:
- net CLK: now also C1.3 (SCLK), C11.5 (SCL), C12.5 (SCL), C17.3 (SCLK), C7.5 (SCL), C8.5 (SCL), D4.1 (K), R25.2; no longer J2.2 (Pin_2)
- net DATA: now also C1.12 (SDAT), C11.7 (SDA), C12.7 (SDA), C17.12 (SDAT), C7.7 (SDA), C8.7 (SDA), D5.1 (K), R26.2; no longer J2.1 (Pin_1)
- net ENinv_1: now also C11.6 (SEN), C7.6 (SEN), D2.1 (K), R23.2; no longer J2.4 (Pin_4)
- net ENinv_2: now also C12.6 (SEN), C8.6 (SEN), D1.1 (K), R22.2; no longer J2.5 (Pin_5)
- net ENser: now also C1.1 (SEN), C17.1 (SEN), D3.1 (K), R24.2; no longer J2.3 (Pin_3)
- net GND: now also D1.2 (A), D2.2 (A), D3.2 (A), D4.2 (A), D5.2 (A)
- new net: J2.1 (Pin_1), R26.1
- new net: J2.2 (Pin_2), R25.1
- new net: J2.3 (Pin_3), R24.1
- new net: J2.4 (Pin_4), R23.1
- new net: J2.5 (Pin_5), R22.1

Commit message: Pre-module commit
Parts:
- added J4, J5: Conn_01x02_Male, Connector_PinHeader_2.54mm:PinHeader_1x02_P2.54mm_Vertical, symbol Connector:Conn_01x02_Male
- L1, L2, L3: footprint Inductor_SMD:L_0603_1608Metric_Pad1.05x0.95mm_HandSolder -> Inductor_SMD:L_0402_1005Metric
Connections:
- net GND: now also J4.2 (Pin_2), J5.2 (Pin_2)
- net SIG_OUT: now reaches C16.1, J3.1 (In)
- net SIG_OUT: now also J5.1 (Pin_1)
- net SIG_IN: now reaches C3.2, J1.1 (In)
- net SIG_IN: now also J4.1 (Pin_1)
Changed lines of the file:
@@
 F 0 "L1" H 3000 3600 50  0000 L CNN
 F 1 "4nH" H 2975 3500 50  0000 L CNN
-F 2 "Inductor_SMD:L_0603_1608Metric_Pad1.05x0.95mm_HandSolder" H 3120 3550 50  0001 C CNN
+F 2 "Inductor_SMD:L_0402_1005Metric" H 3120 3550 50  0001 C CNN
 F 3 "~" H 3120 3550 50  0001 C CNN
 	1    3120 3550
@@
 F 0 "L2" H 5225 3550 50  0000 L CNN
 F 1 "4nH" H 5200 3450 50  0000 L CNN
-F 2 "Inductor_SMD:L_0603_1608Metric_Pad1.05x0.95mm_HandSolder" H 5350 3500 50  0001 C CNN
+F 2 "Inductor_SMD:L_0402_1005Metric" H 5350 3500 50  0001 C CNN
 F 3 "~" H 5350 3500 50  0001 C CNN
 	1    5350 3500
@@
 F 0 "L3" H 7375 3550 50  0000 L CNN
 F 1 "4nH" H 7350 3450 50  0000 L CNN
-F 2 "Inductor_SMD:L_0603_1608Metric_Pad1.05x0.95mm_HandSolder" H 7500 3500 50  0001 C CNN
+F 2 "Inductor_SMD:L_0402_1005Metric" H 7500 3500 50  0001 C CNN
 F 3 "~" H 7500 3500 50  0001 C CNN
 	1    7500 3500
@@
 Wire Wire Line
 	9850 3375 9850 4375
+$Comp
+L Connector:Conn_01x02_Male J4
+U 1 1 5CBAC797
+P 775 4625
+F 0 "J4" H 881 4803 50  0000 C CNN
+F 1 "Conn_01x02_Male" H 881 4712 50  0000 C CNN
+F 2 "Connector_PinHeader_2.54mm:PinHeader_1x02_P2.54mm_Vertical" H 775 4625 50  0001 C CNN
+F 3 "~" H 775 4625 50  0001 C CNN
+	1    775  4625
+	1    0    0    -1
+$EndComp
+$Comp
+L Connector:Conn_01x02_Male J5
+U 1 1 5CBACE4F
+P 10775 4725
+F 0 "J5" H 10881 4903 50  0000 C CNN
+F 1 "Conn_01x02_Male" H 10881 4812 50  0000 C CNN
+F 2 "Connector_PinHeader_2.54mm:PinHeader_1x02_P2.54mm_Vertical" H 10775 4725 50  0001 C CNN
+F 3 "~" H 10775 4725 50  0001 C CNN
+	1    10775 4725
+	-1   0    0    -1
+$EndComp
+Text Label 1100 3450 3    50   ~ 0
+SIG_IN
+Text Label 975  4625 0    50   ~ 0
+SIG_IN
+Text Label 975  4725 0    50   ~ 0
+GND
+Text Label 10550 2850 3    50   ~ 0
+SIG_OUT
+Text Label 10575 4725 2    50   ~ 0
+SIG_OUT
+Text Label 10575 4825 2    50   ~ 0
+GND
 $EndSCHEMATC
